Commit message: go2固定关节加入仿真

File: urdf/urdf/go2w_description_fixed.urdf (robot description, URDF)
Before this commit: robot go2w_description, 35 links, 34 joints
Joints:
- joint FL_calf_joint: axis 0 1 0 -> (none); limit lower=-2.7227 upper=-0.83776 effort=35.55 velocity=20.07 -> (none); origin xyz=0 0 -0.213 rpy=0 0 0 -> xyz=0 0 -0.213 rpy=0 -1.55 0; type revolute -> fixed
- joint FL_calflower1_joint: axis 0 0 0 -> (none)
- joint FL_calflower_joint: axis 0 0 0 -> (none)
- joint FL_foot_motor_joint: axis 0 0 0 -> (none)
- joint FL_hip_joint: axis 1 0 0 -> (none); limit lower=-1.0472 upper=1.0472 effort=23.7 velocity=30.1 -> (none); origin xyz=0.1934 0.0465 0 rpy=0 0 0 -> xyz=0.1934 0.0465 0 rpy=0.08 0 0; type revolute -> fixed
- joint FL_thigh_joint: axis 0 1 0 -> (none); limit lower=-1.5707963267948966 upper=3.4907 effort=23.7 velocity=30.1 -> (none); origin xyz=0 0.0955 0 rpy=0 0 0 -> xyz=0 0.0955 0 rpy=0 0.85 0; type revolute -> fixed
- joint FR_calf_joint: axis 0 1 0 -> (none); limit lower=-2.7227 upper=-0.83776 effort=35.55 velocity=20.07 -> (none); origin xyz=0 0 -0.213 rpy=0 0 0 -> xyz=0 0 -0.213 rpy=0 -1.55 0; type revolute -> fixed
- joint FR_calflower1_joint: axis 0 0 0 -> (none)
- joint FR_calflower_joint: axis 0 0 0 -> (none)
- joint FR_foot_motor_joint: axis 0 0 0 -> (none)
- joint FR_hip_joint: axis 1 0 0 -> (none); limit lower=-1.0472 upper=1.0472 effort=23.7 velocity=30.1 -> (none); origin xyz=0.1934 -0.0465 0 rpy=0 0 0 -> xyz=0.1934 -0.0465 0 rpy=-0.08 0 0; type revolute -> fixed
- joint FR_thigh_joint: axis 0 1 0 -> (none); limit lower=-1.5707963267948966 upper=3.4907 effort=23.7 velocity=30.1 -> (none); origin xyz=0 -0.0955 0 rpy=0 0 0 -> xyz=0 -0.0955 0 rpy=0 0.85 0; type revolute -> fixed
- joint Head_lower_joint: axis 0 0 0 -> (none)
- joint Head_upper_joint: axis 0 0 0 -> (none)
- joint RL_calf_joint: axis 0 1 0 -> (none); limit lower=-2.7227 upper=-0.83776 effort=35.55 velocity=20.07 -> (none); origin xyz=0 0 -0.213 rpy=0 0 0 -> xyz=0 0 -0.213 rpy=0 -1.7 0; type revolute -> fixed
- joint RL_calflower1_joint: axis 0 0 0 -> (none)
- joint RL_calflower_joint: axis 0 0 0 -> (none)
- joint RL_foot_motor_joint: axis 0 0 0 -> (none)
- joint RL_hip_joint: axis 1 0 0 -> (none); limit lower=-1.0472 upper=1.0472 effort=23.7 velocity=30.1 -> (none); origin xyz=-0.1934 0.0465 0 rpy=0 0 0 -> xyz=-0.1934 0.0465 0 rpy=0.08 0 0; type revolute -> fixed
- joint RL_thigh_joint: axis 0 1 0 -> (none); limit lower=-0.5236 upper=4.5379 effort=23.7 velocity=30.1 -> (none); origin xyz=0 0.0955 0 rpy=0 0 0 -> xyz=0 0.0955 0 rpy=0 1.0 0; type revolute -> fixed
- joint RR_calf_joint: axis 0 1 0 -> (none); limit lower=-2.7227 upper=-0.83776 effort=35.55 velocity=20.07 -> (none); origin xyz=0 0 -0.213 rpy=0 0 0 -> xyz=0 0 -0.213 rpy=0 -1.7 0; type revolute -> fixed
- joint RR_calflower1_joint: axis 0 0 0 -> (none)
- joint RR_calflower_joint: axis 0 0 0 -> (none)
- joint RR_foot_motor_joint: axis 0 0 0 -> (none)
- joint RR_hip_joint: axis 1 0 0 -> (none); limit lower=-1.0472 upper=1.0472 effort=23.7 velocity=30.1 -> (none); origin xyz=-0.1934 -0.0465 0 rpy=0 0 0 -> xyz=-0.1934 -0.0465 0 rpy=-0.08 0 0; type revolute -> fixed
- joint RR_thigh_joint: axis 0 1 0 -> (none); limit lower=-0.5236 upper=4.5379 effort=23.7 velocity=30.1 -> (none); origin xyz=0 -0.0955 0 rpy=0 0 0 -> xyz=0 -0.0955 0 rpy=0 1.0 0; type revolute -> fixed
- joint header_lidar_joint: axis 0 0 0 -> (none)
- joint imu_joint: axis 0 0 0 -> (none)
- joint radar_joint: axis 0 0 0 -> (none)
